File: Flight_Controller_V1.kicad_sch (KiCad schematic)
At the start: 0 parts

Commit message: working directory added defs
Parts:
- added AE1: Antenna_Chip, symbol Device:Antenna_Chip
- added C1, C12, C13, C15, C16, C4: 0u1F, Capacitor_SMD:C_0201_0603Metric, symbol Device:C_Small_US
- added C10, C17: 10uF, Capacitor_SMD:C_0201_0603Metric, symbol Device:C_Small_US
- added C11, C14, C9: 1uF, Capacitor_SMD:C_0201_0603Metric, symbol Device:C_Small_US
- added C18, C19: 16pF, Capacitor_SMD:C_0201_0603Metric, symbol Device:C_Small_US
- added C2: 2u2F, Capacitor_SMD:C_0201_0603Metric, symbol Device:C_Small_US
- added C20, C21: 1p4F, Capacitor_SMD:C_0201_0603Metric, symbol Device:C_Small_US
- added C3: 10nF, Capacitor_SMD:C_0402_1005Metric, symbol Device:C_Small_US
- added C5, C6, C8: 100nF, Capacitor_SMD:C_0201_0603Metric, symbol Device:C_Small_US
- added C7: 47pF, Capacitor_SMD:C_0201_0603Metric, symbol Device:C_Small_US
- added J1: U.FL, PCM_JLCPCB:IPEX-SMD_BWIPX-1-001E, symbol PCM_JLCPCB-Extended:RF, Connector, U.FL
- added L1: 27n, Inductor_SMD:L_Neosid_SM-PIC0512H, symbol Device:L_Small
- added L2: 2n, Inductor_SMD:L_0201_0603Metric, symbol Device:L_Small
- added L3: 24n, Inductor_SMD:L_0201_0603Metric, symbol Device:L_Small
- added L4: 2n6, Inductor_SMD:L_0201_0603Metric, symbol Device:L_Small
- added R1, R2: 4k7, Resistor_SMD:R_0201_0603Metric, symbol Device:R
- added R3: 0, Resistor_SMD:R_0201_0603Metric, symbol Device:R_Small
- added R4, R5, R6: 10k, Resistor_SMD:R_0201_0603Metric, symbol Device:R_Small
- added R7: 1k, Resistor_SMD:R_0201_0603Metric, symbol Device:R_Small
- added U1: ICM-42688-P, ICM-42688-P:PQFN50P300X250X97-14N, symbol ICM-42688-P:ICM-42688-P
- added U2: MMC5603NJ, MMC5603NJ:XDCR_MMC5603NJ, symbol MMC5603NJ:MMC5603NJ
- added U3: BMP388, BMP388:PQFN50P200X200X80-10N, symbol BMP388:BMP388
- added U4: NEO-M8N, RF_GPS:ublox_NEO, symbol RF_GPS:NEO-M8N
- added U5: ESP32-C3, Package_DFN_QFN:QFN-32-1EP_5x5mm_P0.5mm_EP3.7x3.7mm, symbol MCU_Espressif:ESP32-C3
- added U6: SX1262IMLTRT, Package_DFN_QFN:QFN-24-1EP_4x4mm_P0.5mm_EP2.6x2.6mm, symbol RF:SX1262IMLTRT
- added U7: W25Q32JVSS, Package_SO:SOIC-8_5.3x5.3mm_P1.27mm, symbol Memory_Flash:W25Q32JVSS
- added X1: 40MHz, 15pF, PCM_JLCPCB:OSC-SMD_4P-L3.2-W2.5-BL_SIT8008BI, symbol PCM_JLCPCB-Extended:Crystal, 40MHz, 15pF
Connections:
- new net: U6.2 (GND), U6.20 (GND), U6.25 (GND), U6.5 (GND), U6.8 (GND)
- new net: R1.2, U2.A2 (SCL)
- new net: R2.2, U2.B2 (SDA)
- new net: R3.1, U4.9 (VCC_RF)
- new net: C7.1, L1.1, R3.2
- new net: AE1.1 (FEED), C20.1, L4.2
- new net: C18.1, L3.1, X1.1 (OSC)
- new net: C19.1, U5.29 (XTAL_N), X1.3 (OSC)
- new net: C21.1, L4.1, U5.1 (LNA_IN)
- new net: C13.1, U5.18 (VDD_SPI)
- new net: C11.1, L2.2, U5.2 (VDD3P3), U5.3 (VDD3P3)
- new net: L3.2, U5.30 (XTAL_P)
- new net: R4.1, U4.14 (LNA_EN)
- new net: R6.1, U4.8 (~{RESET})
- new net: R7.2, U4.3 (TIMEPULSE)
- new net: J1.1 (In), L1.2, U4.11 (RF_IN)
- new net: R5.1, U4.1 (~{SAFEBOOT})
- new net +3.3V: AE1.2 (PCB_Trace), C1.1, C1.2, C10.1, C10.2, C11.2, C12.1, C12.2, C13.2, C14.1, C14.2, C15.1, C15.2, C16.1, C16.2, C17.1, C17.2, C18.2, C19.2, C2.1, C2.2, C20.2, C21.2, C3.1, C3.2, C4.1, C4.2, C5.1, C5.2, C6.1, C6.2, C7.2, C8.1, C8.2, C9.1, C9.2, J1.2 (Ext), L2.1, R1.1, R2.1, R4.2, R5.2, R6.2, R7.1, U1.10 (RESV_10), U1.11 (RESV_11), U1.2 (RESV_2), U1.3 (RESV_3), U1.5 (VDDIO), U1.6 (GND), U1.7 (RESV_7), U1.8 (VDD), U2.A1 (VSA), U2.B1 (VDD), U3.1 (VDDIO), U3.10 (VDD), U3.3 (VSS), U3.8 (VSS), U3.9 (VSS), U4.10 (GND), U4.12 (GND), U4.13 (GND), U4.22 (V_BCKP), U4.23 (VCC), U4.24 (GND), U4.7 (VDD_USB), U5.11 (VDD3P3_RTC), U5.17 (VDD3P3_CPU), U5.31 (VDDA), U5.32 (VDDA), U5.33 (GND), X1.2 (GND), X1.4 (GND)
